Commit message: update for TRON 1

File: src/assets/p1/PF_A.urdf (robot description, URDF)
Before this commit: robot PF_A, 9 links, 8 joints
Links:
- added link contact_L_Link, mass 1e-6
- added link contact_R_Link, mass 1e-6
- added link limx_imu, mass 0.01; visual box size=0.015 0.015 0.004
- link abad_L_Link: mass 1.03648983 -> 1.469; geometry collision cylinder length=0.05 radius=0.05; visual mesh filename=package://assets/p1/meshes/abad_L_Link.STL
- link abad_R_Link: mass 1.03648872 -> 1.469; geometry collision cylinder length=0.05 radius=0.05; visual mesh filename=package://assets/p1/meshes/abad_R_Link.STL
- link base: mass 5.65937068 -> 9.585; geometry collision box size=0.265 0.26 0.18; visual mesh filename=package://assets/p1/meshes/base_Link.STL
- link foot_L_Link: mass 0.14047647 -> 0.18; geometry collision sphere radius=0.032; visual mesh filename=package://assets/p1/meshes/foot_L_Link.STL
- link foot_R_Link: mass 0.14047647 -> 0.18; geometry collision sphere radius=0.032; visual mesh filename=package://assets/p1/meshes/foot_R_Link.STL
- link hip_L_Link: mass 1.73405445 -> 2.3; geometry collision cylinder length=0.18 radius=0.035; visual mesh filename=package://assets/p1/meshes/hip_L_Link.STL
- link hip_R_Link: mass 1.73405240 -> 2.3; geometry collision cylinder length=0.18 radius=0.035; visual mesh filename=package://assets/p1/meshes/hip_R_Link.STL
- link knee_L_Link: mass 0.25930748 -> 0.55; geometry collision cylinder length=0.26 radius=0.015; visual mesh filename=package://assets/p1/meshes/knee_L_Link.STL
- link knee_R_Link: mass 0.25930895 -> 0.55; geometry collision cylinder length=0.26 radius=0.015; visual mesh filename=package://assets/p1/meshes/knee_R_Link.STL
Joints:
- added joint contact_L_Joint: type fixed, parent foot_L_Link, child contact_L_Link, origin xyz=0 0 -0.032 rpy=0 0 0, axis 0 1 0, limit lower=-0 upper=0 effort=60 velocity=50
- added joint contact_R_Joint: type fixed, parent foot_R_Link, child contact_R_Link, origin xyz=0 0 -0.032 rpy=0 0 0, axis 0 1 0, limit lower=-0 upper=0 effort=60 velocity=50
- added joint limx_imu_joint: type fixed, parent base, child limx_imu, origin xyz=0. 0. 0. rpy=0. 0. 0.
- joint abad_L_Joint: limit lower=-0.383972435 upper=0.785398163 effort=40.0 velocity=15.0 -> lower=-0.38397 upper=1.39626 effort=80.0 velocity=15.0; origin xyz=0.0142 0.095 -0.08176 rpy=0 0 0 -> xyz=55.56E-03 105E-03 -260.2E-03 rpy=0 0 0
- joint abad_R_Joint: limit lower=-0.785398163 upper=0.383972435 effort=40.0 velocity=15.0 -> lower=-1.39626 upper=0.38397 effort=80.0 velocity=15.0; origin xyz=0.0142 -0.095 -0.08176 rpy=0 0 0 -> xyz=55.56E-03 -105E-03 -260.2E-03 rpy=0 0 0
- joint foot_L_Joint: origin xyz=0.15 0 -0.29066 rpy=0 0 0 -> xyz=0.150 0 -0.25981 rpy=0 0 0
- joint foot_R_Joint: origin xyz=0.15 0 -0.29066 rpy=0 0 0 -> xyz=0.150 0 -0.25981 rpy=0 0 0
- joint hip_L_Joint: limit lower=-1.047197551 upper=1.483529864 effort=40.0 velocity=15.0 -> lower=-1.012291 upper=1.396263 effort=80.0 velocity=15.0; origin xyz=-0.0802 0.031 0 rpy=0 0 0 -> xyz=-0.077 0.02050 0 rpy=0 0 0
- joint hip_R_Joint: limit lower=-1.483529864 upper=1.047197551 effort=40.0 velocity=15.0 -> lower=-1.396263 upper=1.012291 effort=80.0 velocity=15.0; origin xyz=-0.0802 -0.031 0 rpy=0 0 0 -> xyz=-0.077 -0.02050 0 rpy=0 0 0
- joint knee_L_Joint: limit lower=-1.012290966 upper=1.256637061 effort=40 velocity=15.0 -> lower=-0.872665 upper=1.361357 effort=80 velocity=15; origin xyz=-0.15 -0.021 -0.25981 rpy=0 0 0 -> xyz=-0.1500 -0.02050 -0.25981 rpy=0 0 0
- joint knee_R_Joint: limit lower=-1.256637061 upper=1.012290966 effort=40.0 velocity=15.0 -> lower=-1.361357 upper=0.872665 effort=80 velocity=15; origin xyz=-0.15 0.021 -0.25981 rpy=0 0 0 -> xyz=-0.1500 0.02050 -0.25981 rpy=0 0 0
